File: board/board.sch (EAGLE design)
At the start: 91 parts, among them IC1 LM1117-3.3, IC2 4052SO16, IC3 RASPBERRY_PICOSMD, X1 DF51K-2X4, X10 MOLEX_MICROFIT3.0-2X3, X2 DF51K-2X4, X3 DF51K-2X4, X4 ATF13-2P, X5 DF51K-2X4, X6 ATF13-2P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

Commit message: Version 2.1 board with corrected Pi Power MOSFET and Temperature Connections
Connections:
- removed net N$26: IC2.X1, R40.1, X9.3
- removed net N$34: IC2.X0, R39.1, X9.5
- removed net N$68: IC2.X2, R41.1, X9.1
- new net N$63: IC2.X3, R39.1, X9.5
- new net N$70: IC2.X2, R40.1, X9.3
- new net N$71: IC2.X0, R41.1, X9.1
- net DEBUG_LED: now also IC3.GP21; no longer IC3.GP16
- net N$35: now also IC2.X1; no longer IC2.X3
- net PAS_SEAT_EN: now also IC3.GP16; no longer IC3.GP17
- net PAS_SEAT_LED1: now also IC3.GP19; no longer IC3.GP20
- net PAS_SEAT_LED2: now also IC3.GP18; no longer IC3.GP19
- net PAS_SEAT_LED3: now also IC3.GP17; no longer IC3.GP18
- net PAS_SEAT_SW: now also IC3.GP20; no longer IC3.GP21
Changed lines of the file:
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@@
 <setting verticaltext="up"/>
 </settings>
-<grid distance="0.1" unitdist="inch" unit="inch" style="dots" multiple="1" display="yes" altdistance="0.01" altunitdist="inch" altunit="inch"/>
+<grid distance="0.1" unitdist="inch" unit="inch" style="lines" multiple="1" display="yes" altdistance="0.01" altunitdist="inch" altunit="inch"/>
 <layers>
 <layer number="1" name="Top" color="4" fill="1" visible="no" active="no"/>
@@
 </segment>
 <segment>
-<pinref part="IC3" gate="U$1" pin="GP21"/>
-<wire x1="340.36" y1="99.06" x2="370.84" y2="99.06" width="0.1524" layer="91"/>
-<label x="370.84" y="99.06" size="1.778" layer="95" rot="R180"/>
+<wire x1="340.36" y1="96.52" x2="370.84" y2="96.52" width="0.1524" layer="91"/>
+<pinref part="IC3" gate="U$1" pin="GP20"/>
+<label x="370.84" y="96.52" size="1.778" layer="95" rot="R180"/>
 </segment>
 </net>
@@
 </segment>
 <segment>
-<pinref part="IC3" gate="U$1" pin="GP20"/>
-<wire x1="340.36" y1="96.52" x2="370.84" y2="96.52" width="0.1524" layer="91"/>
-<label x="370.84" y="96.52" size="1.778" layer="95" rot="R180"/>
+<wire x1="340.36" y1="93.98" x2="370.84" y2="93.98" width="0.1524" layer="91"/>
+<pinref part="IC3" gate="U$1" pin="GP19"/>
+<label x="370.84" y="93.98" size="1.778" layer="95" rot="R180"/>
 </segment>
 </net>
@@
 </segment>
 <segment>
-<pinref part="IC3" gate="U$1" pin="GP19"/>
-<wire x1="340.36" y1="93.98" x2="370.84" y2="93.98" width="0.1524" layer="91"/>
-<label x="370.84" y="93.98" size="1.778" layer="95" rot="R180"/>
+<wire x1="340.36" y1="91.44" x2="370.84" y2="91.44" width="0.1524" layer="91"/>
+<pinref part="IC3" gate="U$1" pin="GP18"/>
+<label x="370.84" y="91.44" size="1.778" layer="95" rot="R180"/>
 </segment>
 </net>
@@
 </segment>
 <segment>
-<pinref part="IC3" gate="U$1" pin="GP18"/>
-<wire x1="340.36" y1="91.44" x2="370.84" y2="91.44" width="0.1524" layer="91"/>
-<label x="370.84" y="91.44" size="1.778" layer="95" rot="R180"/>
-</segment>
-</net>
-<net name="N$34" class="0">
-<segment>
-<pinref part="R39" gate="G$1" pin="1"/>
-<pinref part="X9" gate="G$1" pin="5"/>
-<wire x1="48.26" y1="38.1" x2="43.18" y2="38.1" width="0.1524" layer="91"/>
-<pinref part="IC2" gate="G$1" pin="X0"/>
-<wire x1="43.18" y1="38.1" x2="30.48" y2="38.1" width="0.1524" layer="91"/>
-<wire x1="71.12" y1="53.34" x2="43.18" y2="53.34" width="0.1524" layer="91"/>
-<wire x1="43.18" y1="53.34" x2="43.18" y2="38.1" width="0.1524" layer="91"/>
-<junction x="43.18" y="38.1"/>
+<wire x1="340.36" y1="86.36" x2="370.84" y2="86.36" width="0.1524" layer="91"/>
+<pinref part="IC3" gate="U$1" pin="GP17"/>
+<label x="370.84" y="86.36" size="1.778" layer="95" rot="R180"/>
 </segment>
 </net>
@@
 </segment>
 <segment>
-<pinref part="IC3" gate="U$1" pin="GP17"/>
-<wire x1="340.36" y1="86.36" x2="370.84" y2="86.36" width="0.1524" layer="91"/>
-<label x="370.84" y="86.36" size="1.778" layer="95" rot="R180"/>
+<wire x1="340.36" y1="83.82" x2="370.84" y2="83.82" width="0.1524" layer="91"/>
+<pinref part="IC3" gate="U$1" pin="GP16"/>
+<label x="370.84" y="83.82" size="1.778" layer="95" rot="R180"/>
 </segment>
 </net>
@@
 </segment>
 </net>
-<net name="N$68" class="0">
-<segment>
-<pinref part="R41" gate="G$1" pin="1"/>
-<pinref part="X9" gate="G$1" pin="1"/>
-<wire x1="30.48" y1="33.02" x2="38.1" y2="33.02" width="0.1524" layer="91"/>
-<pinref part="IC2" gate="G$1" pin="X2"/>
-<wire x1="38.1" y1="33.02" x2="48.26" y2="33.02" width="0.1524" layer="91"/>
-<wire x1="71.12" y1="48.26" x2="38.1" y2="48.26" width="0.1524" layer="91"/>
-<wire x1="38.1" y1="48.26" x2="38.1" y2="33.02" width="0.1524" layer="91"/>
-<junction x="38.1" y="33.02"/>
-</segment>
-</net>
-<net name="N$26" class="0">
-<segment>
-<pinref part="X9" gate="G$1" pin="3"/>
-<pinref part="R40" gate="G$1" pin="1"/>
-<wire x1="48.26" y1="35.56" x2="40.64" y2="35.56" width="0.1524" layer="91"/>
-<pinref part="IC2" gate="G$1" pin="X1"/>
-<wire x1="40.64" y1="35.56" x2="30.48" y2="35.56" width="0.1524" layer="91"/>
-<wire x1="71.12" y1="50.8" x2="40.64" y2="50.8" width="0.1524" layer="91"/>
-<wire x1="40.64" y1="50.8" x2="40.64" y2="35.56" width="0.1524" layer="91"/>
-<junction x="40.64" y="35.56"/>
-</segment>
-</net>
 <net name="N$35" class="0">
 <segment>
 <pinref part="X9" gate="G$1" pin="7"/>
 <pinref part="R38" gate="G$1" pin="1"/>
-<wire x1="48.26" y1="40.64" x2="45.72" y2="40.64" width="0.1524" layer="91"/>
-<pinref part="IC2" gate="G$1" pin="X3"/>
-<wire x1="45.72" y1="40.64" x2="30.48" y2="40.64" width="0.1524" layer="91"/>
-<wire x1="71.12" y1="45.72" x2="45.72" y2="45.72" width="0.1524" layer="91"/>
-<wire x1="45.72" y1="45.72" x2="45.72" y2="40.64" width="0.1524" layer="91"/>
-<junction x="45.72" y="40.64"/>
+<wire x1="48.26" y1="40.64" x2="43.18" y2="40.64" width="0.1524" layer="91"/>
+<pinref part="IC2" gate="G$1" pin="X1"/>
+<wire x1="43.18" y1="40.64" x2="30.48" y2="40.64" width="0.1524" layer="91"/>
+<wire x1="71.12" y1="50.8" x2="43.18" y2="50.8" width="0.1524" layer="91"/>
+<wire x1="43.18" y1="50.8" x2="43.18" y2="40.64" width="0.1524" layer="91"/>
+<junction x="43.18" y="40.64"/>
 </segment>
 </net>
@@
 </segment>
 <segment>
-<pinref part="IC3" gate="U$1" pin="GP16"/>
-<wire x1="340.36" y1="83.82" x2="370.84" y2="83.82" width="0.1524" layer="91"/>
-<label x="370.84" y="83.82" size="1.778" layer="95" rot="R180"/>
-</segment>
-</net>
+<pinref part="IC3" gate="U$1" pin="GP21"/>
+<wire x1="340.36" y1="99.06" x2="370.84" y2="99.06" width="0.1524" layer="91"/>
+<label x="370.84" y="99.06" size="1.778" layer="95" rot="R180"/>
+</segment>
+</net>
+<net name="N$63" class="0">
+<segment>
+<pinref part="X9" gate="G$1" pin="5"/>
+<pinref part="R39" gate="G$1" pin="1"/>
+<wire x1="48.26" y1="38.1" x2="38.1" y2="38.1" width="0.1524" layer="91"/>
+<pinref part="IC2" gate="G$1" pin="X3"/>
+<wire x1="38.1" y1="38.1" x2="30.48" y2="38.1" width="0.1524" layer="91"/>
+<wire x1="71.12" y1="45.72" x2="38.1" y2="45.72" width="0.1524" layer="91"/>
+<wire x1="38.1" y1="45.72" x2="38.1" y2="38.1" width="0.1524" layer="91"/>
+<junction x="38.1" y="38.1"/>
+</segment>
+</net>
+<net name="N$70" class="0">
+<segment>
+<pinref part="X9" gate="G$1" pin="3"/>
+<pinref part="R40" gate="G$1" pin="1"/>
+<wire x1="48.26" y1="35.56" x2="40.64" y2="35.56" width="0.1524" layer="91"/>
+<pinref part="IC2" gate="G$1" pin="X2"/>
+<wire x1="40.64" y1="35.56" x2="30.48" y2="35.56" width="0.1524" layer="91"/>
+<wire x1="71.12" y1="48.26" x2="40.64" y2="48.26" width="0.1524" layer="91"/>
+<wire x1="40.64" y1="48.26" x2="40.64" y2="35.56" width="0.1524" layer="91"/>
+<junction x="40.64" y="35.56"/>
+</segment>
+</net>
+<net name="N$71" class="0">
+<segment>
+<pinref part="R41" gate="G$1" pin="1"/>
+<pinref part="X9" gate="G$1" pin="1"/>
+<wire x1="30.48" y1="33.02" x2="45.72" y2="33.02" width="0.1524" layer="91"/>
+<pinref part="IC2" gate="G$1" pin="X0"/>
+<wire x1="45.72" y1="33.02" x2="48.26" y2="33.02" width="0.1524" layer="91"/>
+<wire x1="71.12" y1="53.34" x2="45.72" y2="53.34" width="0.1524" layer="91"/>
+<wire x1="45.72" y1="53.34" x2="45.72" y2="33.02" width="0.1524" layer="91"/>
+<junction x="45.72" y="33.02"/>
+</segment>
+</net>

Commit message: Updated board layout with pulldown resistors for N channel MOSFETS
Parts:
- added R45, R46: 560, SMD:RESISTOR0805
- R10, R19, R6: value 120 -> 1k
- R11: value 120 -> 10k
- R14, R15, R22, R23, R8: value 560 -> 120
- R17, R25, R9: value 1k -> 560
- R18: value 120 -> 560
- R26: value (none) -> 560
- R27: value (none) -> 1k
- R30, R31: value 120 -> (none)
- R32, R35: value 1k -> 120
- R34: value 560 -> 1k
- R38: value 10k -> 560
- R39: value 10k -> 1k
- R42, R43: value 560 -> 10k
- R5: value 1k -> 10k
Connections:
- net +12V: now also R17.2, R18.2, R25.2, R26.2, R36.2, R38.1, R39.2, R9.2; no longer R14.2, R15.2, R22.2, R23.2, R34.2, R36.1, R37.2, R8.2
- net +3V3: now also R28.2, R34.2; no longer R26.2, R32.2
- net BATTERY_CHARGE: now also R35.1; no longer R33.1
- net DEBUG_LED: now also R30.2; no longer R28.2
- net DRV_SEAT_EN: now also R15.2; no longer R13.2
- net DRV_SEAT_LED1: now also R12.1; no longer R10.1
- net DRV_SEAT_LED2: now also R13.1; no longer R11.1
- net DRV_SEAT_LED3: now also R14.1; no longer R12.1
- net ENGINE_RUN_OUT: now also R31.2; no longer R29.2
- net GND: now also R11.1, R5.1
- net MIRROR_EN: now also R8.2; no longer R7.2
- net MIRROR_LED1: now also R7.1; no longer R6.1
- net N$10: now also R24.1; no longer R22.1
- net N$11: now also R25.1; no longer R23.1
- net N$12: now also R26.1; no longer R24.1
- net N$15: now also R41.2; no longer R39.2
- net N$16: now also R40.2; no longer R38.2
- net N$24: now also R7.2; no longer R6.2
- net N$25: now also R32.2; no longer R30.2
- net N$27: now also R28.1; no longer R26.1
- net N$28: now also R12.2; no longer R10.2
- net N$29: now also R13.2; no longer R11.2
- net N$3: now also R9.1; no longer R8.1
- net N$30: now also R14.2; no longer R12.2
- net N$31: now also R20.2; no longer R18.2
- net N$32: now also R21.2; no longer R19.2
- net N$33: now also R22.2; no longer R20.2
- net N$35: now also R40.1; no longer R38.1
- net N$37: now also R5.2
- net N$4: now also R36.1; no longer R34.1
- net N$41: now also R10.2, R11.2; no longer R9.2
- net N$42: now also R8.1; no longer R7.1
- net N$43: now also R10.1; no longer R9.1
- net N$44: now also R33.1; no longer R31.1
- net N$45: now also R37.1; no longer R35.1
- net N$46: now also R37.2; no longer R35.2
- net N$47: now also R44.2; no longer R42.2
- net N$48: now also R44.1; no longer R42.1
- net N$49: now also R46.1; no longer R44.1
- net N$5: now also R43.2; no longer R41.2
- net N$50: now also R46.2; no longer R44.2
- net N$51: now also R15.1; no longer R13.1
- net N$52: now also R19.1; no longer R17.1
- net N$53: now also R19.2; no longer R17.2
- net N$54: now also R45.1; no longer R43.1
- net N$55: now also R45.2; no longer R43.2
- net N$56: now also R38.2; no longer R36.2
- net N$57: now also R27.1; no longer R25.1
- net N$58: now also R23.1; no longer R21.1
- net N$59: now also R27.2; no longer R25.2
- net N$6: now also R42.2; no longer R40.2
- net N$60: now also R34.1; no longer R32.1
- net N$61: now also R35.2; no longer R33.2
- net N$62: now also R39.1; no longer R37.1
- net N$63: now also R41.1; no longer R39.1
- net N$64: now also R6.2; no longer R5.2
- net N$66: now also R29.1; no longer R27.1
- net N$67: now also R31.1; no longer R29.1
- net N$69: now also R30.1; no longer R28.1
- net N$7: now also R16.1; no longer R14.1
- net N$70: now also R42.1; no longer R40.1
- net N$71: now also R43.1; no longer R41.1
- net N$8: now also R17.1; no longer R15.1
- net N$9: now also R18.1; no longer R16.1
- net PAS_SEAT_EN: now also R23.2; no longer R21.2
- net PAS_SEAT_LED1: now also R20.1; no longer R18.1
- net PAS_SEAT_LED2: now also R21.1; no longer R19.1
- net PAS_SEAT_LED3: now also R22.1; no longer R20.1
- net USB_POWER: now also R29.2, R6.1; no longer R27.2, R5.1
- net WHEEL_EN: now also R33.2; no longer R31.2
- net WHEEL_LED1: now also R32.1; no longer R30.1
Other:
- moved on the sheet: OK2, OK4, R10, R11, R12, R13, R14, R15, R16, R17, R18, R19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
